File: ThermometerPCB/Mainboard2xAAA/Thermometer.kicad_pcb (KiCad board)
At the start: 2 copper layers, 55 x 39.4 mm, 19 parts, among them J1 DEBUG, J2 LCD, SW1 SW, U1 E18-MS1-PCB, U2 DS18B20, U3 BME280, U4 MAX1678

Commit message: New PCB Uploads
Parts:
- removed REF** (x4): MountingHole_3.2mm_M3, MountingHole:MountingHole_3.2mm_M3
- C3: footprint Capacitor_Tantalum_SMD:CP_EIA-7260-20_AVX-M -> Capacitor_Tantalum_SMD:CP_EIA-3528-15_AVX-H
Routing:
- net GND: track 131.0 -> 132.3 mm
- net +3V3: track 68.0 -> 69.3 mm
