File: ThermometerPCB/eInk_BME280/eInk_BME280.sch (KiCad schematic (older format))
At the start: 19 parts, among them J1 eInk, J2 SPI, Q1 AO3400A

Commit message: New PCB Uploads
Parts:
- removed J2: SPI, symbol Connector_Generic:Conn_01x08
- added C11: 100nF, Capacitor_SMD:C_0603_1608Metric, symbol Device:C
- added J2, J3: SPI1, Connector_PinHeader_1.27mm:PinHeader_1x04_P1.27mm_Vertical, symbol Connector_Generic:Conn_01x04
- added J4: BME280, Connector_PinHeader_1.27mm:PinHeader_1x06_P1.27mm_Vertical, symbol Connector_Generic:Conn_01x06
- added U1: BME280, Package_LGA:Bosch_LGA-8_2.5x2.5mm_P0.65mm_ClockwisePinNumbering, symbol Sensor:BME280
- C1, C10, C2, C3, C4, C5, C6, C7, C8, C9: footprint (none) -> Capacitor_SMD:C_0603_1608Metric
- J1: footprint (none) -> MyLib:FPC-0.5-24P
- L1: footprint CDRH4D18NP100NC -> CDRH4D18NP-2R2NC:CDRH4D18NP100NC
- R1, R2: footprint (none) -> Resistor_SMD:R_0603_1608Metric
Connections:
- net labels added: CS1, MISO, MOSI, P1.0, SCK
- wire segments 58 -> 70
Changed lines of the file:
@@
 F 0 "L1" H 1350 2875 50  0000 C CNN
 F 1 "CDRH4D18NP-10uH 1A" H 1350 2784 50  0000 C CNN
-F 2 "CDRH4D18NP100NC" H 1600 2700 50  0001 L CNN
+F 2 "CDRH4D18NP-2R2NC:CDRH4D18NP100NC" H 1600 2700 50  0001 L CNN
 F 3 "https://componentsearchengine.com/Datasheets/1/CDRH4D18NP-100NC.pdf" H 1600 2600 50  0001 L CNN
 F 4 "Fixed Inductors 2.2uH 1.32A 30% SMD LP INDUCTOR" H 1600 2500 50  0001 L CNN "Description"
@@
 F 0 "J1" H 4780 1842 50  0000 L CNN
 F 1 "eInk" H 4780 1751 50  0000 L CNN
-F 2 "" H 4700 1850 50  0001 C CNN
+F 2 "MyLib:FPC-0.5-24P" H 4700 1850 50  0001 C CNN
 F 3 "~" H 4700 1850 50  0001 C CNN
 	1    4700 1850
@@
 F 0 "C7" V 3548 1150 50  0000 C CNN
 F 1 "1uF" V 3639 1150 50  0000 C CNN
-F 2 "" H 3838 1000 50  0001 C CNN
+F 2 "Capacitor_SMD:C_0603_1608Metric" H 3838 1000 50  0001 C CNN
 F 3 "~" H 3800 1150 50  0001 C CNN
 	1    3800 1150
@@
 F 0 "C4" V 3348 2150 50  0000 C CNN
 F 1 "1uF" V 3439 2150 50  0000 C CNN
-F 2 "" H 3638 2000 50  0001 C CNN
+F 2 "Capacitor_SMD:C_0603_1608Metric" H 3638 2000 50  0001 C CNN
 F 3 "~" H 3600 2150 50  0001 C CNN
 	1    3600 2150
@@
 F 0 "C8" V 3598 2450 50  0000 C CNN
 F 1 "1uF" V 3689 2450 50  0000 C CNN
-F 2 "" H 3888 2300 50  0001 C CNN
+F 2 "Capacitor_SMD:C_0603_1608Metric" H 3888 2300 50  0001 C CNN
 F 3 "~" H 3850 2450 50  0001 C CNN
 	1    3850 2450
@@
 F 0 "C5" V 3348 2750 50  0000 C CNN
 F 1 "1uF" V 3439 2750 50  0000 C CNN
-F 2 "" H 3638 2600 50  0001 C CNN
+F 2 "Capacitor_SMD:C_0603_1608Metric" H 3638 2600 50  0001 C CNN
 F 3 "~" H 3600 2750 50  0001 C CNN
 	1    3600 2750
@@
 F 0 "C10" V 3598 3650 50  0000 C CNN
 F 1 "1uF" V 3689 3650 50  0000 C CNN
-F 2 "" H 3888 3500 50  0001 C CNN
+F 2 "Capacitor_SMD:C_0603_1608Metric" H 3888 3500 50  0001 C CNN
 F 3 "~" H 3850 3650 50  0001 C CNN
 	1    3850 3650
@@
 F 0 "C6" V 3348 3350 50  0000 C CNN
 F 1 "1uF" V 3439 3350 50  0000 C CNN
-F 2 "" H 3638 3200 50  0001 C CNN
+F 2 "Capacitor_SMD:C_0603_1608Metric" H 3638 3200 50  0001 C CNN
 F 3 "~" H 3600 3350 50  0001 C CNN
 	1    3600 3350
@@
 F 0 "C9" V 3598 3050 50  0000 C CNN
 F 1 "1uF" V 3689 3050 50  0000 C CNN
-F 2 "" H 3888 2900 50  0001 C CNN
+F 2 "Capacitor_SMD:C_0603_1608Metric" H 3888 2900 50  0001 C CNN
 F 3 "~" H 3850 3050 50  0001 C CNN
 	1    3850 3050
@@
 F 0 "C1" H 735 2846 50  0000 R CNN
 F 1 "4.7uF" H 735 2755 50  0000 R CNN
-F 2 "" H 888 2650 50  0001 C CNN
+F 2 "Capacitor_SMD:C_0603_1608Metric" H 888 2650 50  0001 C CNN
 F 3 "~" H 850 2800 50  0001 C CNN
 	1    850  2800
@@
 F 0 "R2" H 1920 3396 50  0000 L CNN
 F 1 "3R" H 1920 3305 50  0000 L CNN
-F 2 "" V 1780 3350 50  0001 C CNN
+F 2 "Resistor_SMD:R_0603_1608Metric" V 1780 3350 50  0001 C CNN
 F 3 "~" H 1850 3350 50  0001 C CNN
 	1    1850 3350
@@
 F 0 "R1" H 1470 3396 50  0000 L CNN
 F 1 "10k" H 1470 3305 50  0000 L CNN
-F 2 "" V 1330 3350 50  0001 C CNN
+F 2 "Resistor_SMD:R_0603_1608Metric" V 1330 3350 50  0001 C CNN
 F 3 "~" H 1400 3350 50  0001 C CNN
 	1    1400 3350
@@
 F 0 "C2" H 1735 2296 50  0000 R CNN
 F 1 "4.7uF" H 1735 2205 50  0000 R CNN
-F 2 "" H 1888 2100 50  0001 C CNN
+F 2 "Capacitor_SMD:C_0603_1608Metric" H 1888 2100 50  0001 C CNN
 F 3 "~" H 1850 2250 50  0001 C CNN
 	1    1850 2250
@@
 F 0 "C3" H 2715 2846 50  0000 L CNN
 F 1 "1uF" H 2715 2755 50  0000 L CNN
-F 2 "" H 2638 2650 50  0001 C CNN
+F 2 "Capacitor_SMD:C_0603_1608Metric" H 2638 2650 50  0001 C CNN
 F 3 "~" H 2600 2800 50  0001 C CNN
 	1    2600 2800
@@
 Text Label 2950 1600 2    50   ~ 0
 PREVGL
-$Comp
-L Connector_Generic:Conn_01x08 J2
-U 1 1 60903E0C
-P 900 1250
-F 0 "J2" H 818 1767 50  0000 C CNN
-F 1 "SPI" H 818 1676 50  0000 C CNN
-F 2 "" H 900 1250 50  0001 C CNN
-F 3 "~" H 900 1250 50  0001 C CNN
-	1    900  1250
+Wire Wire Line
+	1300 850  1050 850
+Wire Wire Line
+	1300 950  1050 950
+Wire Wire Line
+	1300 1050 1050 1050
+Wire Wire Line
+	1300 1150 1050 1150
+Text Label 1300 850  2    50   ~ 0
+BUSY
+Text Label 1300 950  2    50   ~ 0
+RES
+Text Label 1300 1050 2    50   ~ 0
+DC
+Text Label 1300 1150 2    50   ~ 0
+CS
+$Comp
+L Connector_Generic:Conn_01x04 J3
+U 1 1 609DB327
+P 850 1600
+F 0 "J3" H 768 1917 50  0000 C CNN
+F 1 "SPI1" H 768 1826 50  0000 C CNN
+F 2 "Connector_PinHeader_1.27mm:PinHeader_1x04_P1.27mm_Vertical" H 850 1600 50  0001 C CNN
+F 3 "~" H 850 1600 50  0001 C CNN
+	1    850  1600
 	-1   0    0    -1
 $EndComp
 Wire Wire Line
-	1350 950  1100 950
-Wire Wire Line
-	1350 1050 1100 1050
-Wire Wire Line
-	1350 1150 1100 1150
-Wire Wire Line
-	1350 1250 1100 1250
-Wire Wire Line
-	1350 1350 1100 1350
-Wire Wire Line
-	1350 1450 1100 1450
-Wire Wire Line
-	1350 1550 1100 1550
-Wire Wire Line
-	1350 1650 1100 1650
-Text Label 1350 950  2    50   ~ 0
-BUSY
-Text Label 1350 1050 2    50   ~ 0
-RES
-Text Label 1350 1150 2    50   ~ 0
-DC
-Text Label 1350 1250 2    50   ~ 0
-CS
-Text Label 1350 1350 2    50   ~ 0
+	1300 1500 1050 1500
+Wire Wire Line
+	1300 1600 1050 1600
+$Comp
+L power:GND #PWR0101
+U 1 1 609E1FD0
+P 1300 1700
+F 0 "#PWR0101" H 1300 1450 50  0001 C CNN
+F 1 "GND" V 1305 1572 50  0000 R CNN
+F 2 "" H 1300 1700 50  0001 C CNN
+F 3 "" H 1300 1700 50  0001 C CNN
+	1    1300 1700
+	0    -1   1    0
+$EndComp
+$Comp
+L power:+3.3V #PWR0102
+U 1 1 609E2BE0
+P 1300 1800
+F 0 "#PWR0102" H 1300 1650 50  0001 C CNN
+F 1 "+3.3V" V 1315 1928 50  0000 L CNN
+F 2 "" H 1300 1800 50  0001 C CNN
+F 3 "" H 1300 1800 50  0001 C CNN
+	1    1300 1800
+	0    1    1    0
+$EndComp
+Wire Wire Line
+	1300 1700 1050 1700
+Wire Wire Line
+	1300 1800 1050 1800
+Text Label 1300 1500 2    50   ~ 0
 SCLK
-Text Label 1350 1450 2    50   ~ 0
+Text Label 1300 1600 2    50   ~ 0
 SDI
 $Comp
+L Connector_Generic:Conn_01x04 J2
+U 1 1 609E9B19
+P 850 950
+F 0 "J2" H 768 1267 50  0000 C CNN
+F 1 "SPI1" H 768 1176 50  0000 C CNN
+F 2 "Connector_PinHeader_1.27mm:PinHeader_1x04_P1.27mm_Vertical" H 850 950 50  0001 C CNN
+F 3 "~" H 850 950 50  0001 C CNN
+	1    850  950
+	-1   0    0    -1
+$EndComp
+$Comp
+L Sensor:BME280 U1
+U 1 1 609F93A8
+P 2850 5400
+F 0 "U1" H 2421 5446 50  0000 R CNN
+F 1 "BME280" H 2421 5355 50  0000 R CNN
+F 2 "Package_LGA:Bosch_LGA-8_2.5x2.5mm_P0.65mm_ClockwisePinNumbering" H 4350 4950 50  0001 C CNN
+F 3 "https://ae-bst.resource.bosch.com/media/_tech/media/datasheets/BST-BME280-DS002.pdf" H 2850 5200 50  0001 C CNN
+	1    2850 5400
+	1    0    0    -1
+$EndComp
+Wire Wire Line
+	3200 4800 2950 4800
+Connection ~ 2950 4800
+Wire Wire Line
+	2950 4800 2750 4800
+Wire Wire Line
+	3700 5100 3450 5100
+Wire Wire Line
+	3700 5300 3450 5300
+Wire Wire Line
+	3700 5500 3450 5500
+Wire Wire Line
+	3700 5700 3450 5700
+$Comp
+L power:GND #PWR04
+U 1 1 60A01FA3
+P 2750 6000
+F 0 "#PWR04" H 2750 5750 50  0001 C CNN
+F 1 "GND" H 2755 5827 50  0000 C CNN
+F 2 "" H 2750 6000 50  0001 C CNN
+F 3 "" H 2750 6000 50  0001 C CNN
+	1    2750 6000
+	1    0    0    -1
+$EndComp
+$Comp
+L power:GND #PWR012
+U 1 1 60A02831
+P 2950 6000
+F 0 "#PWR012" H 2950 5750 50  0001 C CNN
+F 1 "GND" H 2955 5827 50  0000 C CNN
+F 2 "" H 2950 6000 50  0001 C CNN
+F 3 "" H 2950 6000 50  0001 C CNN
+	1    2950 6000
+	1    0    0    -1
+$EndComp
+$Comp
+L Device:C C11
+U 1 1 60A03350
+P 1950 4950
+F 0 "C11" H 2065 4996 50  0000 L CNN
+F 1 "100nF" H 2065 4905 50  0000 L CNN
+F 2 "Capacitor_SMD:C_0603_1608Metric" H 1988 4800 50  0001 C CNN
+F 3 "~" H 1950 4950 50  0001 C CNN
+	1    1950 4950
+	1    0    0    -1
+$EndComp
+$Comp
 L power:GND #PWR03
-U 1 1 60911295
-P 1350 1550
-F 0 "#PWR03" H 1350 1300 50  0001 C CNN
-F 1 "GND" V 1355 1422 50  0000 R CNN
-F 2 "" H 1350 1550 50  0001 C CNN
-F 3 "" H 1350 1550 50  0001 C CNN
-	1    1350 1550
-	0    -1   1    0
-$EndComp
-$Comp
-L power:+3.3V #PWR04
-U 1 1 60911B18
-P 1350 1650
-F 0 "#PWR04" H 1350 1500 50  0001 C CNN
-F 1 "+3.3V" V 1365 1778 50  0000 L CNN
-F 2 "" H 1350 1650 50  0001 C CNN
-F 3 "" H 1350 1650 50  0001 C CNN
-	1    1350 1650
-	0    1    1    0
-$EndComp
+U 1 1 60A03E36
+P 1950 5100
+F 0 "#PWR03" H 1950 4850 50  0001 C CNN
+F 1 "GND" H 1955 4927 50  0000 C CNN
+F 2 "" H 1950 5100 50  0001 C CNN
+F 3 "" H 1950 5100 50  0001 C CNN
+	1    1950 5100
+	1    0    0    -1
+$EndComp
+Wire Wire Line
+	1950 4800 2750 4800
+Connection ~ 2750 4800
+Text Label 3200 4800 2    50   ~ 0
+P1.0
+Text Label 3700 5100 2    50   ~ 0
+MISO
+Text Label 3700 5300 2    50   ~ 0
+SCK
+Text Label 3700 5500 2    50   ~ 0
+MOSI
+Text Label 3700 5700 2    50   ~ 0
+CS1
+$Comp
+L Connector_Generic:Conn_01x06 J4
+U 1 1 60A07A99
+P 4900 5200
+F 0 "J4" H 4980 5192 50  0000 L CNN
+F 1 "BME280" H 4980 5101 50  0000 L CNN
+F 2 "Connector_PinHeader_1.27mm:PinHeader_1x06_P1.27mm_Vertical" H 4900 5200 50  0001 C CNN
+F 3 "~" H 4900 5200 50  0001 C CNN
+	1    4900 5200
+	1    0    0    -1
+$EndComp
+Wire Wire Line
+	4450 5000 4700 5000
+Wire Wire Line
+	4450 5100 4700 5100
+Wire Wire Line
+	4450 5200 4700 5200
+Wire Wire Line
+	4450 5300 4700 5300
+Wire Wire Line
+	4450 5400 4700 5400
+$Comp
+L power:GND #PWR013
+U 1 1 60A11CDC
+P 4700 5500
+F 0 "#PWR013" H 4700 5250 50  0001 C CNN
+F 1 "GND" H 4705 5327 50  0000 C CNN
+F 2 "" H 4700 5500 50  0001 C CNN
+F 3 "" H 4700 5500 50  0001 C CNN
+	1    4700 5500
+	0    1    1    0
+$EndComp
+Text Label 4450 5000 0    50   ~ 0
+P1.0
+Text Label 4450 5100 0    50   ~ 0
+MISO
+Text Label 4450 5200 0    50   ~ 0
+SCK
+Text Label 4450 5300 0    50   ~ 0
+MOSI
+Text Label 4450 5400 0    50   ~ 0
+CS1
 $EndSCHEMATC
