File: ThermometerPCB/Mainboard_NRF52833_CR2450/Thermometer.kicad_pcb (KiCad board)
At the start: 2 copper layers, 50.5 x 38.3 mm, 21 parts, among them J1 Debug, J2 LCD, J3 LCD, J4 Sensor, SW1 SW, U1 E73-2G4M08S1E, Y1 32.768kHz

Commit message: NRF52833 board  update
Parts:
- Y1: footprint Crystal:Crystal_SMD_0603-2Pin_6.0x3.5mm -> Crystal:Crystal_SMD_MicroCrystal_CC8V-T1A-2Pin_2.0x1.2mm_HandSoldering
Routing:
- net Net-(C3-Pad1): track 10.3 -> 11.4 mm
- net Net-(C4-Pad1): track 11.4 -> 12.2 mm
