File: ThermometerPCB/Mainboard_NRF52833_CR2450/Thermometer.sch (KiCad schematic (older format))
At the start: 21 parts, among them J1 Debug, J2 LCD, J3 LCD, J4 Sensor, SW1 SW, U1 E73-2G4M08S1E, Y1 32.768kHz

Commit message: NRF52833 board  update
Parts:
- Y1: footprint Crystal:Crystal_SMD_0603-2Pin_6.0x3.5mm -> Crystal:Crystal_SMD_MicroCrystal_CC8V-T1A-2Pin_2.0x1.2mm_HandSoldering
Changed lines of the file:
@@
 F 0 "Y1" H 4400 4018 50  0000 C CNN
 F 1 "32.768kHz" H 4400 3927 50  0000 C CNN
-F 2 "Crystal:Crystal_SMD_0603-2Pin_6.0x3.5mm" H 4400 3750 50  0001 C CNN
+F 2 "Crystal:Crystal_SMD_MicroCrystal_CC8V-T1A-2Pin_2.0x1.2mm_HandSoldering" H 4400 3750 50  0001 C CNN
 F 3 "~" H 4400 3750 50  0001 C CNN
 	1    4400 3750
