File: ThermometerPCB/eInk_Si7021/eInk_Si7021.kicad_pcb (KiCad board)
At the start: 2 copper layers, 50.5 x 38.3 mm, 23 parts, among them J1 eInk, J2 SPI1, J3 SPI1, J4 Si7021, Q1 AO3400A, U1 Si7021-A20

Commit message: NRF52833 board  update
Changed lines of the file:
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@@
-(kicad_pcb (version 20171130) (host pcbnew "(5.1.10)-1")
+(kicad_pcb (version 20171130) (host pcbnew "(5.1.8)-1")
   (general
     (thickness 1.6)
@@
     (add_net "Net-(U1-Pad7)")
   )
+  (module MyLib:FPC-0.5-24P (layer B.Cu)
+    (at 72.7456 77.0126 90)
+    (attr smd)
+    (fp_text reference J1 (at 0.2411 2.3114) (layer B.SilkS)
+      (effects (font (size 1 1) (thickness 0.15)) (justify mirror))
+    )
+    (fp_text value eInk (at 0 -2.925 -90) (layer B.Fab)
+      (effects (font (size 1 1) (thickness 0.15)) (justify mirror))
+    )
+    (fp_line (start -6 0.805) (end 6 0.805) (layer B.SilkS) (width 0.12))
+    (fp_line (start -6 -0.805) (end 6 -0.805) (layer B.SilkS) (width 0.12))
+    (fp_line (start -6 -0.805) (end -6 -3.945) (layer B.SilkS) (width 0.12))
+    (fp_line (start 6 -0.805) (end 6 -3.945) (layer B.SilkS) (width 0.12))
+    (fp_line (start -6 -3.945) (end -10.5 -3.945) (layer B.SilkS) (width 0.12))
+    (fp_line (start 6 -3.945) (end 10.5 -3.945) (layer B.SilkS) (width 0.12))
+    (fp_line (start -10.5 -3.945) (end -10.5 -0.585) (layer B.SilkS) (width 0.12))
+    (fp_line (start 10.5 -3.945) (end 10.5 -0.585) (layer B.SilkS) (width 0.12))
+    (fp_line (start -10.5 -0.585) (end -6 -0.585) (layer B.SilkS) (width 0.12))
+    (fp_line (start 10.5 -0.585) (end 6 -0.585) (layer B.SilkS) (width 0.12))
+    (fp_line (start -6 -0.585) (end -6 0.805) (layer B.SilkS) (width 0.12))
+    (fp_line (start 6 -0.585) (end 6 0.805) (layer B.SilkS) (width 0.12))
+    (fp_line (start -10.79 1.05) (end 10.79 1.05) (layer B.CrtYd) (width 0.05))
+    (fp_line (start 10.79 1.05) (end 10.79 -4.2) (layer B.CrtYd) (width 0.05))
+    (fp_line (start -10.79 -4.2) (end 10.79 -4.2) (layer B.CrtYd) (width 0.05))
+    (fp_line (start -10.79 1.05) (end -10.79 -4.2) (layer B.CrtYd) (width 0.05))
+    (pad 0 smd rect (at 8.29 -2.325 90) (size 4 3) (layers B.Cu B.Paste B.Mask))
+    (pad 0 smd rect (at -8.29 -2.325 90) (size 4 3) (layers B.Cu B.Paste B.Mask))
+    (pad 24 smd rect (at -5.75 0 90) (size 0.3 1.25) (layers B.Cu B.Paste B.Mask)
+      (net 13 /VCOM))
+    (pad 23 smd rect (at -5.25 0 90) (size 0.3 1.25) (layers B.Cu B.Paste B.Mask)
+      (net 2 /PREVGL))
+    (pad 22 smd rect (at -4.75 0 90) (size 0.3 1.25) (layers B.Cu B.Paste B.Mask)
+      (net 12 "Net-(C9-Pad1)"))
+    (pad 21 smd rect (at -4.25 0 90) (size 0.3 1.25) (layers B.Cu B.Paste B.Mask)
+      (net 4 /PREVGH))
+    (pad 20 smd rect (at -3.75 0 90) (size 0.3 1.25) (layers B.Cu B.Paste B.Mask)
+      (net 8 "Net-(C5-Pad1)"))
+    (pad 19 smd rect (at -3.25 0 90) (size 0.3 1.25) (layers B.Cu B.Paste B.Mask)
+      (net 24 "Net-(J1-Pad19)"))
+    (pad 18 smd rect (at -2.75 0 90) (size 0.3 1.25) (layers B.Cu B.Paste B.Mask)
+      (net 11 "Net-(C8-Pad1)"))
+    (pad 17 smd rect (at -2.25 0 90) (size 0.3 1.25) (layers B.Cu B.Paste B.Mask)
+      (net 3 GND))
+    (pad 16 smd rect (at -1.75 0 90) (size 0.3 1.25) (layers B.Cu B.Paste B.Mask)
+      (net 9 +3V3))
+    (pad 15 smd rect (at -1.25 0 90) (size 0.3 1.25) (layers B.Cu B.Paste B.Mask)
+      (net 9 +3V3))
+    (pad 14 smd rect (at -0.75 0 90) (size 0.3 1.25) (layers B.Cu B.Paste B.Mask)
+      (net 23 /SDI))
+    (pad 13 smd rect (at -0.25 0 90) (size 0.3 1.25) (layers B.Cu B.Paste B.Mask)
+      (net 22 /SCLK))
+    (pad 12 smd rect (at 0.25 0 90) (size 0.3 1.25) (layers B.Cu B.Paste B.Mask)
+      (net 21 /CS))
+    (pad 11 smd rect (at 0.75 0 90) (size 0.3 1.25) (layers B.Cu B.Paste B.Mask)
+      (net 20 /DC))
+    (pad 10 smd rect (at 1.25 0 90) (size 0.3 1.25) (layers B.Cu B.Paste B.Mask)
+      (net 19 /RES))
+    (pad 9 smd rect (at 1.75 0 90) (size 0.3 1.25) (layers B.Cu B.Paste B.Mask)
+      (net 18 /BUSY))
+    (pad 8 smd rect (at 2.25 0 90) (size 0.3 1.25) (layers B.Cu B.Paste B.Mask)
+      (net 3 GND))
+    (pad 7 smd rect (at 2.75 0 90) (size 0.3 1.25) (layers B.Cu B.Paste B.Mask)
+      (net 17 "Net-(J1-Pad7)"))
+    (pad 6 smd rect (at 3.25 0 90) (size 0.3 1.25) (layers B.Cu B.Paste B.Mask)
+      (net 16 "Net-(J1-Pad6)"))
+    (pad 5 smd rect (at 3.75 0 90) (size 0.3 1.25) (layers B.Cu B.Paste B.Mask)
+      (net 10 "Net-(C7-Pad1)"))
+    (pad 4 smd rect (at 4.25 0 90) (size 0.3 1.25) (layers B.Cu B.Paste B.Mask)
+      (net 15 "Net-(J1-Pad4)"))
+    (pad 3 smd rect (at 4.75 0 90) (size 0.3 1.25) (layers B.Cu B.Paste B.Mask)
+      (net 7 /RESE))
+    (pad 2 smd rect (at 5.25 0 90) (size 0.3 1.25) (layers B.Cu B.Paste B.Mask)
+      (net 6 /GDR))
+    (pad 1 smd rect (at 5.75 0 90) (size 0.3 1.25) (layers B.Cu B.Paste B.Mask)
+      (net 14 "Net-(J1-Pad1)"))
+  )
   (module Diode_SMD:D_SOD-123 (layer B.Cu)
     (at 81.788 88.9762 270)
@@
     )
   )
-  (module MyLib:FPC-0.5-24P (layer B.Cu)
-    (at 72.7456 77.0126 90)
-    (attr smd)
-    (fp_text reference J1 (at 0 -1.775 -90) (layer B.SilkS)
-      (effects (font (size 1 1) (thickness 0.15)) (justify mirror))
-    )
-    (fp_text value eInk (at 0 -2.925 -90) (layer B.Fab)
-      (effects (font (size 1 1) (thickness 0.15)) (justify mirror))
-    )
-    (fp_line (start -6 0.805) (end 6 0.805) (layer B.SilkS) (width 0.12))
-    (fp_line (start -6 -0.805) (end 6 -0.805) (layer B.SilkS) (width 0.12))
-    (fp_line (start -6 -0.805) (end -6 -3.945) (layer B.SilkS) (width 0.12))
-    (fp_line (start 6 -0.805) (end 6 -3.945) (layer B.SilkS) (width 0.12))
-    (fp_line (start -6 -3.945) (end -8.65 -3.945) (layer B.SilkS) (width 0.12))
-    (fp_line (start 6 -3.945) (end 8.65 -3.945) (layer B.SilkS) (width 0.12))
-    (fp_line (start -8.65 -3.945) (end -8.65 -0.585) (layer B.SilkS) (width 0.12))
-    (fp_line (start 8.65 -3.945) (end 8.65 -0.585) (layer B.SilkS) (width 0.12))
-    (fp_line (start -8.65 -0.585) (end -6 -0.585) (layer B.SilkS) (width 0.12))
-    (fp_line (start 8.65 -0.585) (end 6 -0.585) (layer B.SilkS) (width 0.12))
-    (fp_line (start -6 -0.585) (end -6 0.805) (layer B.SilkS) (width 0.12))
-    (fp_line (start 6 -0.585) (end 6 0.805) (layer B.SilkS) (width 0.12))
-    (fp_line (start -8.9 1.05) (end 8.9 1.05) (layer B.CrtYd) (width 0.05))
-    (fp_line (start 8.9 1.05) (end 8.9 -4.2) (layer B.CrtYd) (width 0.05))
-    (fp_line (start -8.9 -4.2) (end 8.9 -4.2) (layer B.CrtYd) (width 0.05))
-    (fp_line (start -8.9 1.05) (end -8.9 -4.2) (layer B.CrtYd) (width 0.05))
-    (pad 1 smd rect (at 5.75 0 90) (size 0.3 1.25) (layers B.Cu B.Paste B.Mask)
-      (net 14 "Net-(J1-Pad1)"))
-    (pad 2 smd rect (at 5.25 0 90) (size 0.3 1.25) (layers B.Cu B.Paste B.Mask)
-      (net 6 /GDR))
-    (pad 3 smd rect (at 4.75 0 90) (size 0.3 1.25) (layers B.Cu B.Paste B.Mask)
-      (net 7 /RESE))
-    (pad 4 smd rect (at 4.25 0 90) (size 0.3 1.25) (layers B.Cu B.Paste B.Mask)
-      (net 15 "Net-(J1-Pad4)"))
-    (pad 5 smd rect (at 3.75 0 90) (size 0.3 1.25) (layers B.Cu B.Paste B.Mask)
-      (net 10 "Net-(C7-Pad1)"))
-    (pad 6 smd rect (at 3.25 0 90) (size 0.3 1.25) (layers B.Cu B.Paste B.Mask)
-      (net 16 "Net-(J1-Pad6)"))
-    (pad 7 smd rect (at 2.75 0 90) (size 0.3 1.25) (layers B.Cu B.Paste B.Mask)
-      (net 17 "Net-(J1-Pad7)"))
-    (pad 8 smd rect (at 2.25 0 90) (size 0.3 1.25) (layers B.Cu B.Paste B.Mask)
-      (net 3 GND))
-    (pad 9 smd rect (at 1.75 0 90) (size 0.3 1.25) (layers B.Cu B.Paste B.Mask)
-      (net 18 /BUSY))
-    (pad 10 smd rect (at 1.25 0 90) (size 0.3 1.25) (layers B.Cu B.Paste B.Mask)
-      (net 19 /RES))
-    (pad 11 smd rect (at 0.75 0 90) (size 0.3 1.25) (layers B.Cu B.Paste B.Mask)
-      (net 20 /DC))
-    (pad 12 smd rect (at 0.25 0 90) (size 0.3 1.25) (layers B.Cu B.Paste B.Mask)
-      (net 21 /CS))
-    (pad 13 smd rect (at -0.25 0 90) (size 0.3 1.25) (layers B.Cu B.Paste B.Mask)
-      (net 22 /SCLK))
-    (pad 14 smd rect (at -0.75 0 90) (size 0.3 1.25) (layers B.Cu B.Paste B.Mask)
-      (net 23 /SDI))
-    (pad 15 smd rect (at -1.25 0 90) (size 0.3 1.25) (layers B.Cu B.Paste B.Mask)
-      (net 9 +3V3))
-    (pad 16 smd rect (at -1.75 0 90) (size 0.3 1.25) (layers B.Cu B.Paste B.Mask)
-      (net 9 +3V3))
-    (pad 17 smd rect (at -2.25 0 90) (size 0.3 1.25) (layers B.Cu B.Paste B.Mask)
-      (net 3 GND))
-    (pad 18 smd rect (at -2.75 0 90) (size 0.3 1.25) (layers B.Cu B.Paste B.Mask)
-      (net 11 "Net-(C8-Pad1)"))
-    (pad 19 smd rect (at -3.25 0 90) (size 0.3 1.25) (layers B.Cu B.Paste B.Mask)
-      (net 24 "Net-(J1-Pad19)"))
-    (pad 20 smd rect (at -3.75 0 90) (size 0.3 1.25) (layers B.Cu B.Paste B.Mask)
-      (net 8 "Net-(C5-Pad1)"))
-    (pad 21 smd rect (at -4.25 0 90) (size 0.3 1.25) (layers B.Cu B.Paste B.Mask)
-      (net 4 /PREVGH))
-    (pad 22 smd rect (at -4.75 0 90) (size 0.3 1.25) (layers B.Cu B.Paste B.Mask)
-      (net 12 "Net-(C9-Pad1)"))
-    (pad 23 smd rect (at -5.25 0 90) (size 0.3 1.25) (layers B.Cu B.Paste B.Mask)
-      (net 2 /PREVGL))
-    (pad 24 smd rect (at -5.75 0 90) (size 0.3 1.25) (layers B.Cu B.Paste B.Mask)
-      (net 13 /VCOM))
-    (pad 0 smd rect (at -7.29 -2.325 90) (size 2 3) (layers B.Cu B.Paste B.Mask))
-    (pad 0 smd rect (at 7.29 -2.325 90) (size 2 3) (layers B.Cu B.Paste B.Mask))
-  )
   (module Capacitor_SMD:C_0603_1608Metric (layer B.Cu)
     (at 80.137 81.2422 270)
@@
     (tags Inductor)
     (attr smd)
-    (fp_text reference L1 (at 0 0 90) (layer B.SilkS)
+    (fp_text reference L1 (at -0.1524 4.6486 90) (layer B.SilkS)
       (effects (font (size 1.27 1.27) (thickness 0.254)) (justify mirror))
     )
